File: lazyboy36/PCB/lazyboy36.kicad_pcb (KiCad board)
At the start: 2 copper layers, 73 parts, among them SW1 Switch-NoLED, SW10 Switch-NoLED, SW11 Switch-NoLED, SW12 Switch-NoLED, SW13 Switch-NoLED, SW14 Switch-NoLED, SW15 Switch-NoLED, SW16 Switch-NoLED, SW17 Switch-NoLED, SW18 Switch-NoLED, SW19 Switch-NoLED, SW2 Switch-NoLED, SW20 Switch-NoLED, SW21 Switch-NoLED, SW22 Switch-NoLED, SW23 Switch-NoLED, SW24 Switch-NoLED, SW25 Switch-NoLED, SW26 Switch-NoLED, SW27 Switch-NoLED, SW28 Switch-NoLED, SW29 Switch-NoLED, SW3 Switch-NoLED, SW30 Switch-NoLED, SW31 Switch-NoLED, SW32 Switch-NoLED, SW33 Switch-NoLED, SW34 Switch-NoLED, SW35 Switch-NoLED, SW36 Switch-NoLED, SW4 Switch-NoLED, SW5 Switch-NoLED, SW6 Switch-NoLED, SW7 Switch-NoLED, SW8 Switch-NoLED, SW9 Switch-NoLED, U1 ProMicro_RP2040_R

Commit message: 설계 진행
Parts:
- moved D34 30.7 mm to (170.1, 143.0), turned to 40 degrees
- moved D33 28.0 mm to (127.0, 143.4), turned to 140 degrees
- moved SW34 27.7 mm to (173.3, 146.8), turned to 40 degrees
- moved SW33 25.3 mm to (123.8, 147.2), turned to -40 degrees
- moved D35 22.4 mm to (189.7, 130.4), turned to 25 degrees
- moved SW35 20.3 mm to (191.8, 134.9), turned to 25 degrees
- moved D36 17.7 mm to (211.4, 124.0), turned to 10 degrees
- moved D32 16.9 mm to (105.4, 130.7), turned to 155 degrees
- moved D8 16.8 mm to (212.7, 57.2), turned to 15 degrees
- moved D6 16.8 mm to (177.7, 73.9), turned to 15 degrees
- moved SW36 16.8 mm to (212.2, 129.0), turned to 10 degrees
- moved SW32 16.5 mm to (105.3, 135.2), turned to -25 degrees
- moved D9 16.2 mm to (232.4, 57.1), turned to 15 degrees
- moved SW6 15.7 mm to (179.0, 78.7), turned to 15 degrees
- moved SW8 15.7 mm to (214.0, 62.1), turned to 15 degrees
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Routing:
- net Net-(D1-A): track 12.6 -> 0.00 mm
- net Net-(D2-A): track 12.6 -> 0.00 mm

Commit message: 낄낄
Parts:
- moved D34 0.34 mm to (170.1, 143.4)
- moved SW34 0.34 mm to (173.3, 147.2)
- moved D35 0.30 mm to (189.7, 130.7)
- moved SW35 0.30 mm to (191.8, 135.2)
- moved D10 0.27 mm to (253.9, 64.1)
- moved D16 0.27 mm to (182.7, 92.5)
- moved D19 0.27 mm to (237.3, 75.8)
- moved D20 0.27 mm to (258.8, 82.5)
- moved D26 0.27 mm to (187.6, 110.9)
- moved D27 0.27 mm to (205.5, 104.1)
- moved D28 0.27 mm to (222.6, 94.3)
- moved D29 0.27 mm to (242.3, 94.2)
- moved D30 0.27 mm to (263.8, 100.9)
- moved D6 0.27 mm to (177.7, 74.1)
- moved SW10 0.27 mm to (255.2, 68.9)
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
Commit message: 업뎁
Parts:
- D1, D10, D11, D12, D13, D14, D15, D16, D17, D18, D19, D2, D20, D21, D22, D23, D24, D25, D26, D27, D28, D29, D3, D30, D31, D32, D33, D34, D35, D36, D4, D5, D6, D7, D8, D9: footprint KBD:D3_SMD -> KBD:D3_TH_SMD_v2
- moved D32 2.00 mm to (107.4, 130.7), turned to -25 degrees
- turned D1 to -15 degrees
- turned D11 to -15 degrees
- turned D12 to -15 degrees
- turned D13 to -15 degrees
- turned D14 to -15 degrees
- turned D15 to -15 degrees
- turned D2 to -15 degrees
- turned D21 to -15 degrees
- turned D22 to -15 degrees
- turned D23 to -15 degrees
- turned D24 to -15 degrees
- turned D25 to -15 degrees
- turned D3 to -15 degrees
- turned D31 to -10 degrees
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Routing:
- net ROW1: track 0.00 -> 172.7 mm
- net ROW0: track 0.00 -> 172.5 mm
- net ROW2: track 0.00 -> 171.8 mm
- net ROW3: track 0.00 -> 143.1 mm
- net COL5: track 0.00 -> 83.8 mm
- net COL6: track 0.00 -> 78.1 mm
- net COL2: track 0.00 -> 76.7 mm
- net COL7: track 0.00 -> 75.4 mm
- net COL4: track 0.00 -> 74.6 mm
- net COL3: track 0.00 -> 71.7 mm
- net COL8: track 0.00 -> 40.9 mm
- net COL1: track 0.00 -> 40.9 mm
- net COL9: track 0.00 -> 40.9 mm
- net COL0: track 0.00 -> 40.9 mm
- net Net-(D34-A): track 0.00 -> 12.6 mm
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
Commit message: fsdf
Parts:
- moved SW31 9.29 mm to (75.6, 129.3)
- moved D31 9.29 mm to (76.5, 124.4)
- moved SW36 9.16 mm to (221.4, 129.3)
- moved D36 9.16 mm to (220.5, 124.4)
- moved D3 8.95 mm to (75.6, 55.7)
- moved SW13 8.95 mm to (69.4, 78.9)
- moved SW23 8.95 mm to (64.5, 97.3)
- moved D12 8.95 mm to (51.0, 74.0)
- moved SW12 8.95 mm to (49.7, 78.8)
- moved SW22 8.95 mm to (44.8, 97.2)
- moved D14 8.95 mm to (87.8, 83.9)
- moved D15 8.95 mm to (105.7, 90.7)
- moved D2 8.95 mm to (55.9, 55.6)
- moved D22 8.95 mm to (46.1, 92.4)
- moved D24 8.95 mm to (82.9, 102.3)
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Routing:
- net COL0: track 40.9 -> 209.1 mm, vias 0 -> 2
- net COL1: track 40.9 -> 165.2 mm, vias 0 -> 2
- net ROW0: track 172.5 -> 296.0 mm, vias 0 -> 2
- net COL9: track 40.9 -> 155.5 mm, vias 0 -> 1
- net ROW2: track 171.8 -> 273.0 mm
- net ROW1: track 172.7 -> 269.9 mm, vias 0 -> 2
- net COL2: track 76.7 -> 170.5 mm, vias 0 -> 2
- net COL8: track 40.9 -> 132.2 mm, vias 0 -> 1
- net COL7: track 75.4 -> 153.2 mm, vias 0 -> 1
- net ROW3: track 143.1 -> 216.5 mm, vias 0 -> 1
- net COL3: track 71.7 -> 139.4 mm, vias 0 -> 2
- net COL6: track 78.1 -> 131.9 mm, vias 0 -> 1
- net COL5: track 83.8 -> 133.8 mm, vias 0 -> 1
- net COL4: track 74.6 -> 123.1 mm, vias 0 -> 2
- net Net-(D35-A): track 11.9 -> 13.6 mm
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- added copper zone on B.Cu, net (none)
- added copper zone on F.Cu, net (none)
Other:
- board outline added: 282.6 x 144.3 mm

Commit message: 설계 거의 완료
Other:
- board size 282.6 x 144.3 mm -> 275.6 x 113.1 mm

Commit message: 설계변경, 불필요 배선 삭제
Routing:
- net COL0: track 209.1 -> 171.0 mm
- net ROW3: track 216.5 -> 242.1 mm
- net ROW0: track 296.0 -> 298.7 mm
- net COL2: track 170.5 -> 168.7 mm
Changed lines of the file:
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@@
-	)
-	(segment
-		(start 72.635019 54.819246)
-		(end 72.735893 54.92012)
-		(width 0.2)
-		(layer "F.Cu")
-		(net 1)
 	)
 	(segment
@@
 	)
 	(segment
+		(start 84 62)
+		(end 82.5 60.5)
+		(width 0.2)
+		(layer "F.Cu")
+		(net 1)
+	)
+	(segment
 		(start 107.725935 71.542606)
 		(end 113.67011 71.542606)
@@
 	)
 	(segment
+		(start 82.5 60.5)
+		(end 82.5 57.337566)
+		(width 0.2)
+		(layer "F.Cu")
+		(net 1)
+	)
+	(segment
+		(start 60.819246 54.819246)
+		(end 62 56)
+		(width 0.2)
+		(layer "F.Cu")
+		(net 1)
+	)
+	(segment
+		(start 53.040911 54.819246)
+		(end 60.819246 54.819246)
+		(width 0.2)
+		(layer "F.Cu")
+		(net 1)
+	)
+	(segment
+		(start 72.735893 54.92012)
+		(end 80.082554 54.92012)
+		(width 0.2)
+		(layer "F.Cu")
+		(net 1)
+	)
+	(segment
 		(start 218.559402 56.372294)
 		(end 218.458529 56.473167)
@@
 	)
 	(segment
-		(start 80.082554 54.92012)
-		(end 89.842686 64.680252)
+		(start 82.5 57.337566)
+		(end 80.082554 54.92012)
 		(width 0.2)
 		(layer "F.Cu")
@@
 	)
 	(segment
+		(start 71.656013 56)
+		(end 72.735893 54.92012)
+		(width 0.2)
+		(layer "F.Cu")
+		(net 1)
+	)
+	(segment
 		(start 245.521294 56.372294)
 		(end 238.153511 56.372294)
@@
 	)
 	(segment
-		(start 72.735893 54.92012)
-		(end 80.082554 54.92012)
-		(width 0.2)
-		(layer "F.Cu")
-		(net 1)
-	)
-	(segment
 		(start 139.1 102.3734)
 		(end 140.9364 100.537)
@@
 	)
 	(segment
-		(start 53.040911 54.819246)
-		(end 72.635019 54.819246)
+		(start 87.162434 62)
+		(end 84 62)
+		(width 0.2)
+		(layer "F.Cu")
+		(net 1)
+	)
+	(segment
+		(start 89.842686 64.680252)
+		(end 87.162434 62)
 		(width 0.2)
 		(layer "F.Cu")
@@
 		(start 201.352737 66.233299)
 		(end 194.490382 73.095654)
+		(width 0.2)
+		(layer "F.Cu")
+		(net 1)
+	)
+	(segment
+		(start 62 56)
+		(end 71.656013 56)
 		(width 0.2)
 		(layer "F.Cu")
@@
 	)
 	(segment
+		(start 155.8 109.05)
+		(end 158.234314 109.05)
+		(width 0.2)
+		(layer "F.Cu")
+		(net 13)
+	)
+	(segment
+		(start 159.481742 110.297427)
+		(end 172.797427 110.297427)
+		(width 0.2)
+		(layer "F.Cu")
+		(net 13)
+	)
+	(segment
 		(start 210.610068 131.9)
 		(end 217.563912 124.946156)
@@
 	)
 	(segment
-		(start 119.446951 142.255784)
-		(end 116.203266 142.255784)
-		(width 0.2)
-		(layer "F.Cu")
-		(net 13)
-	)
-	(segment
-		(start 152.652735 109.05)
-		(end 155.8 109.05)
+		(start 177.2 145.104087)
+		(end 176.191445 146.112642)
 		(width 0.2)
 		(layer "F.Cu")
@@
 	)
 	(segment
+		(start 172.797427 110.297427)
+		(end 177.2 114.7)
+		(width 0.2)
+		(layer "F.Cu")
+		(net 13)
+	)
+	(segment
 		(start 176.191445 146.112642)
 		(end 177.904087 144.4)
@@
 	)
 	(segment
-		(start 152.652735 109.05)
-		(end 119.446951 142.255784)
-		(width 0.2)
-		(layer "F.Cu")
-		(net 13)
-	)
-	(segment
 		(start 196.047884 131.9)
 		(end 210.610068 131.9)
@@
 	)
 	(segment
-		(start 177.2 145.104087)
-		(end 176.191445 146.112642)
+		(start 121.45 109.05)
+		(end 116.203266 114.296734)
 		(width 0.2)
 		(layer "F.Cu")
@@
 	)
 	(segment
-		(start 177.2 130.45)
-		(end 177.2 145.104087)
+		(start 155.8 109.05)
+		(end 121.45 109.05)
 		(width 0.2)
 		(layer "F.Cu")
@@
 	)
 	(segment
-		(start 155.8 109.05)
-		(end 177.2 130.45)
+		(start 158.234314 109.05)
+		(end 159.481742 110.297427)
+		(width 0.2)
+		(layer "F.Cu")
+		(net 13)
+	)
+	(segment
+		(start 116.203266 114.296734)
+		(end 116.203266 142.255784)
 		(width 0.2)
 		(layer "F.Cu")
@@
 		(start 195.434338 132.515662)
 		(end 195.434338 132.514546)
+		(width 0.2)
+		(layer "F.Cu")
+		(net 13)
+	)
+	(segment
+		(start 177.2 114.7)
+		(end 177.2 145.104087)
 		(width 0.2)
 		(layer "F.Cu")
@@
 	)
 	(segment
-		(start 19.191074 87.936715)
-		(end 14.260572 106.337602)
-		(width 0.2)
-		(layer "B.Cu")
-		(net 41)
-	)
-	(segment
 		(start 24.121576 69.535827)
 		(end 24.121576 83.006212)
@@
 		(start 123.377006 91.35)
 		(end 137.45 91.35)
-		(width 0.2)
-		(layer "B.Cu")
-		(net 41)
-	)
-	(segment
-		(start 24.121577 69.535828)
-		(end 19.191074 87.936715)
 		(width 0.2)
 		(layer "B.Cu")
@@
 	)
 	(segment
-		(start 65.323275 76.446477)
-		(end 60.392771 81.376981)
-		(width 0.2)
-		(layer "B.Cu")
-		(net 43)
-	)
-	(segment
-		(start 60.392771 94.847365)
-		(end 55.462268 99.777868)
+		(start 69.5 125.477)
+		(end 69.5 110.5)
+		(width 0.2)
+		(layer "B.Cu")
+		(net 43)
+	)
+	(segment
+		(start 64 108)
+		(end 61 105)
+		(width 0.2)
+		(layer "B.Cu")
+		(net 43)
+	)
+	(segment
+		(start 66.834931 128.142069)
+		(end 69.5 125.477)
 		(width 0.2)
 		(layer "B.Cu")
@@
 	)
 	(segment
+		(start 67 108)
+		(end 64 108)
+		(width 0.2)
+		(layer "B.Cu")
+		(net 43)
+	)
+	(segment
 		(start 123.177 92.917)
 		(end 123.21 92.917)
@@
 	)
 	(segment
+		(start 55.462268 99.777868)
+		(end 60.392771 94.847365)
+		(width 0.2)
+		(layer "B.Cu")
+		(net 43)
+	)
+	(segment
+		(start 55.462268 102.785268)
+		(end 55.462268 99.777868)
+		(width 0.2)
+		(layer "B.Cu")
+		(net 43)
+	)
+	(segment
+		(start 65.323275 76.446477)
+		(end 65.323275 70.8)
+		(width 0.2)
+		(layer "B.Cu")
+		(net 43)
+	)
+	(segment
 		(start 60.392771 81.376981)
-		(end 60.392771 94.847365)
-		(width 0.2)
-		(layer "B.Cu")
-		(net 43)
-	)
-	(segment
-		(start 66.834931 128.142069)
-		(end 70.127 124.85)
-		(width 0.2)
-		(layer "B.Cu")
-		(net 43)
-	)
-	(segment
-		(start 61.627 103.95)
-		(end 56.627 103.95)
-		(width 0.2)
-		(layer "B.Cu")
-		(net 43)
-	)
-	(segment
-		(start 56.627 103.95)
-		(end 55.462268 102.785268)
-		(width 0.2)
-		(layer "B.Cu")
-		(net 43)
-	)
-	(segment
-		(start 70.127 124.85)
-		(end 70.127 108.95)
+		(end 65.323275 76.446477)
 		(width 0.2)
 		(layer "B.Cu")
@@
 	)
 	(segment
-		(start 70.127 108.95)
-		(end 67.427 106.25)
-		(width 0.2)
-		(layer "B.Cu")
-		(net 43)
-	)
-	(segment
 		(start 140.3084 92.917)
 		(end 123.41 92.917)
@@
 	)
 	(segment
-		(start 55.462268 102.785268)
-		(end 55.462268 99.777868)
-		(width 0.2)
-		(layer "B.Cu")
-		(net 43)
-	)
-	(segment
 		(start 66.834931 132.575503)
 		(end 66.834931 132.575504)
@@
 	)
 	(segment
+		(start 57.677 105)
+		(end 55.462268 102.785268)
+		(width 0.2)
+		(layer "B.Cu")
+		(net 43)
+	)
+	(segment
 		(start 66.834931 132.575503)
 		(end 66.834931 128.142069)
@@
 	)
 	(segment
-		(start 63.927 106.25)
-		(end 61.627 103.95)
-		(width 0.2)
-		(layer "B.Cu")
-		(net 43)
-	)
-	(segment
-		(start 65.323275 70.8)
-		(end 65.323275 76.446477)
-		(width 0.2)
-		(layer "B.Cu")
-		(net 43)
-	)
-	(segment
-		(start 67.427 106.25)
-		(end 63.927 106.25)
+		(start 69.5 110.5)
+		(end 67 108)
+		(width 0.2)
+		(layer "B.Cu")
+		(net 43)
+	)
+	(segment
+		(start 60.392771 94.847365)
+		(end 60.392771 81.376981)
+		(width 0.2)
+		(layer "B.Cu")
+		(net 43)
+	)
+	(segment
+		(start 61 105)
+		(end 57.677 105)
 		(width 0.2)
 		(layer "B.Cu")
@@
 		(polygon
 			(pts
-				(xy -25.775583 -11.845324) (xy 307.674417 14.354676) (xy 300.774417 183.204676) (xy -2.375583 182.554676)
+				(xy 25.5 40) (xy 84 46) (xy 119.5 59.5) (xy 149 64) (xy 182 59.5) (xy 217.5 44.5) (xy 274 42.5)
+				(xy 292.5 112) (xy 179 169) (xy 165 153) (xy 131 153) (xy 115.5 168) (xy 4.5 113.5)
 			)
 		)
