File: lazyboy36/PCB/lazyboy36.kicad_sch (KiCad schematic)
At the start: 73 parts, among them SW1 Switch-NoLED, SW10 Switch-NoLED, SW11 Switch-NoLED, SW12 Switch-NoLED, SW13 Switch-NoLED, SW14 Switch-NoLED, SW15 Switch-NoLED, SW16 Switch-NoLED, SW17 Switch-NoLED, SW18 Switch-NoLED, SW19 Switch-NoLED, SW2 Switch-NoLED, SW20 Switch-NoLED, SW21 Switch-NoLED, SW22 Switch-NoLED, SW23 Switch-NoLED, SW24 Switch-NoLED, SW25 Switch-NoLED, SW26 Switch-NoLED, SW27 Switch-NoLED, SW28 Switch-NoLED, SW29 Switch-NoLED, SW3 Switch-NoLED, SW30 Switch-NoLED, SW31 Switch-NoLED, SW32 Switch-NoLED, SW33 Switch-NoLED, SW34 Switch-NoLED, SW35 Switch-NoLED, SW36 Switch-NoLED, SW4 Switch-NoLED, SW5 Switch-NoLED, SW6 Switch-NoLED, SW7 Switch-NoLED, SW8 Switch-NoLED, SW9 Switch-NoLED, U1 ProMicro_RP2040_R

Commit message: 업뎁
Parts:
- D1, D10, D11, D12, D13, D14, D15, D16, D17, D18, D19, D2, D20, D21, D22, D23, D24, D25, D26, D27, D28, D29, D3, D30, D31, D32, D33, D34, D35, D36, D4, D5, D6, D7, D8, D9: footprint KBD:D3_SMD -> KBD:D3_TH_SMD_v2

Commit message: 설계 중단
Parts:
- SW1, SW10, SW11, SW12, SW13, SW14, SW15, SW16, SW17, SW18, SW19, SW2, SW20, SW21, SW22, SW23, SW24, SW25, SW26, SW27, SW28, SW29, SW3, SW30, SW31, SW32, SW33, SW34, SW35, SW36, SW4, SW5, SW6, SW7, SW8, SW9: footprint KBD:SW_Gateron_LowProfile_HotSwap_PTH -> KBD:SW_Gateron_LowProfile_HotSwap_PTH_복사
Changed lines of the file:
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@@
 			)
 		)
-		(property "Footprint" "KBD:SW_Gateron_LowProfile_HotSwap_PTH"
+		(property "Footprint" "KBD:SW_Gateron_LowProfile_HotSwap_PTH_복사"
 			(at 170.5356 85.725 0)
 			(effects
@@
 			)
 		)
-		(property "Footprint" "KBD:SW_Gateron_LowProfile_HotSwap_PTH"
+		(property "Footprint" "KBD:SW_Gateron_LowProfile_HotSwap_PTH_복사"
 			(at 159.1056 85.725 0)
 			(effects
@@
 			)
 		)
-		(property "Footprint" "KBD:SW_Gateron_LowProfile_HotSwap_PTH"
+		(property "Footprint" "KBD:SW_Gateron_LowProfile_HotSwap_PTH_복사"
 			(at 193.3956 103.505 0)
 			(effects
@@
 			)
 		)
-		(property "Footprint" "KBD:SW_Gateron_LowProfile_HotSwap_PTH"
+		(property "Footprint" "KBD:SW_Gateron_LowProfile_HotSwap_PTH_복사"
 			(at 147.6756 85.725 0)
 			(effects
@@
 			)
 		)
-		(property "Footprint" "KBD:SW_Gateron_LowProfile_HotSwap_PTH"
+		(property "Footprint" "KBD:SW_Gateron_LowProfile_HotSwap_PTH_복사"
 			(at 193.3956 67.945 0)
 			(effects
@@
 			)
 		)
-		(property "Footprint" "KBD:SW_Gateron_LowProfile_HotSwap_PTH"
+		(property "Footprint" "KBD:SW_Gateron_LowProfile_HotSwap_PTH_복사"
 			(at 136.2456 85.725 0)
 			(effects
@@
 			)
 		)
-		(property "Footprint" "KBD:SW_Gateron_LowProfile_HotSwap_PTH"
+		(property "Footprint" "KBD:SW_Gateron_LowProfile_HotSwap_PTH_복사"
 			(at 124.8156 67.945 0)
 			(effects
@@
 			)
 		)
-		(property "Footprint" "KBD:SW_Gateron_LowProfile_HotSwap_PTH"
+		(property "Footprint" "KBD:SW_Gateron_LowProfile_HotSwap_PTH_복사"
 			(at 204.8256 85.725 0)
 			(effects
@@
 			)
 		)
-		(property "Footprint" "KBD:SW_Gateron_LowProfile_HotSwap_PTH"
+		(property "Footprint" "KBD:SW_Gateron_LowProfile_HotSwap_PTH_복사"
 			(at 204.8256 67.945 0)
 			(effects
@@
 			)
 		)
-		(property "Footprint" "KBD:SW_Gateron_LowProfile_HotSwap_PTH"
+		(property "Footprint" "KBD:SW_Gateron_LowProfile_HotSwap_PTH_복사"
 			(at 216.2556 67.945 0)
 			(effects
@@
 			)
 		)
-		(property "Footprint" "KBD:SW_Gateron_LowProfile_HotSwap_PTH"
+		(property "Footprint" "KBD:SW_Gateron_LowProfile_HotSwap_PTH_복사"
 			(at 159.1056 67.945 0)
 			(effects
@@
 			)
 		)
-		(property "Footprint" "KBD:SW_Gateron_LowProfile_HotSwap_PTH"
+		(property "Footprint" "KBD:SW_Gateron_LowProfile_HotSwap_PTH_복사"
 			(at 147.6756 67.945 0)
 			(effects
@@
 			)
 		)
-		(property "Footprint" "KBD:SW_Gateron_LowProfile_HotSwap_PTH"
+		(property "Footprint" "KBD:SW_Gateron_LowProfile_HotSwap_PTH_복사"
 			(at 113.3856 67.945 0)
 			(effects
@@
 			)
 		)
-		(property "Footprint" "KBD:SW_Gateron_LowProfile_HotSwap_PTH"
+		(property "Footprint" "KBD:SW_Gateron_LowProfile_HotSwap_PTH_복사"
 			(at 170.5356 103.505 0)
 			(effects
@@
 			)
 		)
-		(property "Footprint" "KBD:SW_Gateron_LowProfile_HotSwap_PTH"
+		(property "Footprint" "KBD:SW_Gateron_LowProfile_HotSwap_PTH_복사"
 			(at 124.8156 85.725 0)
 			(effects
@@
 			)
 		)
-		(property "Footprint" "KBD:SW_Gateron_LowProfile_HotSwap_PTH"
+		(property "Footprint" "KBD:SW_Gateron_LowProfile_HotSwap_PTH_복사"
 			(at 159.1056 103.505 0)
 			(effects
@@
 			)
 		)
-		(property "Footprint" "KBD:SW_Gateron_LowProfile_HotSwap_PTH"
+		(property "Footprint" "KBD:SW_Gateron_LowProfile_HotSwap_PTH_복사"
 			(at 181.9656 67.945 0)
 			(effects
@@
 			)
 		)
-		(property "Footprint" "KBD:SW_Gateron_LowProfile_HotSwap_PTH"
+		(property "Footprint" "KBD:SW_Gateron_LowProfile_HotSwap_PTH_복사"
 			(at 113.3856 50.165 0)
 			(effects
@@
 			)
 		)
-		(property "Footprint" "KBD:SW_Gateron_LowProfile_HotSwap_PTH"
+		(property "Footprint" "KBD:SW_Gateron_LowProfile_HotSwap_PTH_복사"
 			(at 216.2556 85.725 0)
 			(effects
@@
 			)
 		)
-		(property "Footprint" "KBD:SW_Gateron_LowProfile_HotSwap_PTH"
+		(property "Footprint" "KBD:SW_Gateron_LowProfile_HotSwap_PTH_복사"
 			(at 147.6756 103.505 0)
 			(effects
@@
 			)
 		)
-		(property "Footprint" "KBD:SW_Gateron_LowProfile_HotSwap_PTH"
+		(property "Footprint" "KBD:SW_Gateron_LowProfile_HotSwap_PTH_복사"
 			(at 193.3956 50.165 0)
 			(effects
@@
 			)
 		)
-		(property "Footprint" "KBD:SW_Gateron_LowProfile_HotSwap_PTH"
+		(property "Footprint" "KBD:SW_Gateron_LowProfile_HotSwap_PTH_복사"
 			(at 181.9656 85.725 0)
 			(effects
@@
 			)
 		)
-		(property "Footprint" "KBD:SW_Gateron_LowProfile_HotSwap_PTH"
+		(property "Footprint" "KBD:SW_Gateron_LowProfile_HotSwap_PTH_복사"
 			(at 170.5356 50.165 0)
 			(effects
@@
 			)
 		)
-		(property "Footprint" "KBD:SW_Gateron_LowProfile_HotSwap_PTH"
+		(property "Footprint" "KBD:SW_Gateron_LowProfile_HotSwap_PTH_복사"
 			(at 216.2556 50.165 0)
 			(effects
@@
 			)
 		)
-		(property "Footprint" "KBD:SW_Gateron_LowProfile_HotSwap_PTH"
+		(property "Footprint" "KBD:SW_Gateron_LowProfile_HotSwap_PTH_복사"
 			(at 124.8156 50.165 0)
 			(effects
@@
 			)
 		)
-		(property "Footprint" "KBD:SW_Gateron_LowProfile_HotSwap_PTH"
+		(property "Footprint" "KBD:SW_Gateron_LowProfile_HotSwap_PTH_복사"
 			(at 204.8256 50.165 0)
 			(effects
@@
 			)
 		)
-		(property "Footprint" "KBD:SW_Gateron_LowProfile_HotSwap_PTH"
+		(property "Footprint" "KBD:SW_Gateron_LowProfile_HotSwap_PTH_복사"
 			(at 136.2456 67.945 0)
 			(effects
@@
 			)
 		)
-		(property "Footprint" "KBD:SW_Gateron_LowProfile_HotSwap_PTH"
+		(property "Footprint" "KBD:SW_Gateron_LowProfile_HotSwap_PTH_복사"
 			(at 170.5356 67.945 0)
 			(effects
@@
 			)
 		)
-		(property "Footprint" "KBD:SW_Gateron_LowProfile_HotSwap_PTH"
+		(property "Footprint" "KBD:SW_Gateron_LowProfile_HotSwap_PTH_복사"
 			(at 136.2456 50.165 0)
 			(effects
@@
 			)
 		)
-		(property "Footprint" "KBD:SW_Gateron_LowProfile_HotSwap_PTH"
+		(property "Footprint" "KBD:SW_Gateron_LowProfile_HotSwap_PTH_복사"
 			(at 113.3856 85.725 0)
 			(effects
@@
 			)
 		)
-		(property "Footprint" "KBD:SW_Gateron_LowProfile_HotSwap_PTH"
+		(property "Footprint" "KBD:SW_Gateron_LowProfile_HotSwap_PTH_복사"
 			(at 159.1056 50.165 0)
 			(effects
@@
 			)
 		)
-		(property "Footprint" "KBD:SW_Gateron_LowProfile_HotSwap_PTH"
+		(property "Footprint" "KBD:SW_Gateron_LowProfile_HotSwap_PTH_복사"
 			(at 193.3956 85.725 0)
 			(effects
@@
 			)
 		)
-		(property "Footprint" "KBD:SW_Gateron_LowProfile_HotSwap_PTH"
+		(property "Footprint" "KBD:SW_Gateron_LowProfile_HotSwap_PTH_복사"
 			(at 181.9656 50.165 0)
 			(effects
@@
 			)
 		)
-		(property "Footprint" "KBD:SW_Gateron_LowProfile_HotSwap_PTH"
+		(property "Footprint" "KBD:SW_Gateron_LowProfile_HotSwap_PTH_복사"
 			(at 181.9656 103.505 0)
 			(effects
@@
 			)
 		)
-		(property "Footprint" "KBD:SW_Gateron_LowProfile_HotSwap_PTH"
+		(property "Footprint" "KBD:SW_Gateron_LowProfile_HotSwap_PTH_복사"
 			(at 136.2456 103.505 0)
 			(effects
@@
 			)
 		)
-		(property "Footprint" "KBD:SW_Gateron_LowProfile_HotSwap_PTH"
+		(property "Footprint" "KBD:SW_Gateron_LowProfile_HotSwap_PTH_복사"
 			(at 147.6756 50.165 0)
 			(effects
